File: V2/DB15_Switch/DB15_Switch/DB15_Switch.sch (KiCad schematic (older format))
At the start: 35 parts, among them J1 DB15_Male_HighDensity_Mountin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, U1 CH340C, U2 SM420561N, U3 STI3508, U4 ATmega328P-A, Y1 Crystal_GND24

Commit message: update
Parts:
- removed R10: 10K, Resistor_SMD:R_0805_2012Metric, symbol 0805:R
- added U2: HDSP-A151, Display_7Segment:7SegmentLED_LTS6760_LTS6780, symbol Display_Character:HDSP-A151
- renumbered U2 to U?
Connections:
- net +5V: now also U3.4 (EN), U2.1 (CA), U2.6 (CA); no longer U?.3 (CC), U?.8 (CC)
- net A0: now also J1.13; no longer J1.4
- net A1: now also J1.14; no longer J1.5
- net A2: now also J1.12; no longer J1.7
- net A3: now also J1.11; no longer J1.8
- net A4: now also J1.8; no longer J1.10
- net A5: now also J1.7; no longer J1.11
- net A6: now also J1.5; no longer J1.12
- net A7: now also J1.4; no longer J1.13
- net D10: now also RN1.3 (R3.1); no longer RN1.4 (R4.1)
- net D11: now also RN1.2 (R2.1); no longer RN1.3 (R3.1)
- net D12: now also RN1.1 (R1.1); no longer RN1.2 (R2.1)
- net D13: now also J1.10; no longer RN1.1 (R1.1)
- net D2: now also J1.1; no longer U3.4 (EN)
- net D3: now also J1.2; no longer J1.1
- net D4: now also J1.3; no longer J1.2
- net D5: now also RN1.8 (R8.1); no longer J1.3
- net D6: now also RN1.7 (R7.1); no longer RN1.8 (R8.1)
- net D7: now also RN1.6 (R6.1); no longer RN1.7 (R7.1)
- net D8: now also RN1.5 (R5.1); no longer RN1.6 (R6.1)
- net D9: now also RN1.4 (R4.1); no longer RN1.5 (R5.1)
- net at RN1.13 (R4.2): now also U2.2 (F); no longer U?.1 (E)
- net at RN1.12 (R5.2): now also U2.10 (A); no longer U?.10 (G)
- net at RN1.14 (R3.2): now also U2.3 (G); no longer U?.2 (D)
- net at RN1.15 (R2.2): now also U2.5 (D); no longer U?.4 (C)
- net at RN1.16 (R1.2): now also U2.4 (E); no longer U?.5 (DP)
- net at RN1.11 (R6.2): now also U2.9 (B); no longer U?.6 (B)
- net at RN1.10 (R7.2): now also U2.7 (DP); no longer U?.7 (A)
- net at RN1.9 (R8.2): now also U2.8 (C); no longer U?.9 (F)
- no-connect marks 9 -> 8
Other:
- moved on the sheet: U?
Changed lines of the file:
@@
 	7550 1750 7550 1850
 Wire Wire Line
+	7550 1950 7300 1950
+Wire Wire Line
 	7300 1850 7550 1850
+Connection ~ 7550 1850
+Wire Wire Line
+	7550 1850 7550 1950
 $Comp
 L 0805:C C6
@@
 Wire Wire Line
 	800  5900 800  5550
+Text Label 1050 5250 2    50   ~ 0
+D3
+Text Label 1050 5050 2    50   ~ 0
+D4
+Text Label 2350 5500 2    50   ~ 0
+D5
+Text Label 2350 5400 2    50   ~ 0
+D6
+Text Label 2350 5300 2    50   ~ 0
+D7
+Text Label 2350 5100 2    50   ~ 0
+D9
 Text Label 1050 5450 2    50   ~ 0
-D3
-Text Label 1050 5250 2    50   ~ 0
-D4
-Text Label 1050 5050 2    50   ~ 0
-D5
-Text Label 2350 5500 2    50   ~ 0
-D6
-Text Label 2350 5400 2    50   ~ 0
-D7
+D2
 Text Label 2350 5200 2    50   ~ 0
-D9
-Text Label 7300 1950 0    50   ~ 0
-D2
-Text Label 2350 5300 2    50   ~ 0
 D8
-Text Label 2350 5100 2    50   ~ 0
+Text Label 2350 5000 2    50   ~ 0
 D10
+Text Label 2350 4800 2    50   ~ 0
+D12
+Text Label 1050 4750 2    50   ~ 0
+D13
 Text Label 2350 4900 2    50   ~ 0
-D12
-Text Label 2350 4800 2    50   ~ 0
-D13
-Text Label 2350 5000 2    50   ~ 0
 D11
+Text Label 1650 5050 0    50   ~ 0
+A0
+Text Label 1650 4850 0    50   ~ 0
+A1
+Text Label 1650 5250 0    50   ~ 0
+A2
+Text Label 1650 5450 0    50   ~ 0
+A3
+Text Label 1050 5150 2    50   ~ 0
+A4
+Text Label 1050 5350 2    50   ~ 0
+A5
+Text Label 1050 4650 2    50   ~ 0
+A6
 Text Label 1050 4850 2    50   ~ 0
-A0
-Text Label 1050 4650 2    50   ~ 0
-A1
-Text Label 1050 5350 2    50   ~ 0
-A2
-Text Label 1050 5150 2    50   ~ 0
-A3
-Text Label 1050 4750 2    50   ~ 0
-A4
-Text Label 1650 5450 0    50   ~ 0
-A5
-Text Label 1650 5250 0    50   ~ 0
-A6
-Text Label 1650 5050 0    50   ~ 0
 A7
 Text Label 1650 4650 0    50   ~ 0
@@
 	-1   0    0    1
 $EndComp
+Wire Wire Line
+	2650 5300 3400 5300
+Wire Wire Line
+	3400 5300 3400 4900
+Wire Wire Line
+	3400 4900 3550 4900
+Wire Wire Line
+	3550 4800 3050 4800
+Wire Wire Line
+	3050 4800 3050 5200
+Wire Wire Line
+	3050 5200 2650 5200
+Wire Wire Line
+	2650 4800 3000 4800
+Wire Wire Line
+	3000 4800 3000 5100
+Wire Wire Line
+	2650 4900 3250 4900
+Wire Wire Line
+	3250 4900 3250 5100
+Wire Wire Line
+	3150 5150 2750 5150
+Wire Wire Line
+	2750 5150 2750 5100
+Wire Wire Line
+	2750 5100 2650 5100
+Wire Wire Line
+	2650 5000 2900 5000
+Wire Wire Line
+	2900 5000 2900 5400
+Wire Wire Line
+	2650 5500 3450 5500
+Wire Wire Line
+	3450 5500 3450 5000
+Wire Wire Line
+	3450 5000 3550 5000
+Wire Wire Line
+	3550 5500 3500 5500
+Wire Wire Line
+	3500 5500 3500 5450
+Wire Wire Line
+	3500 5450 2700 5450
+Wire Wire Line
+	2700 5450 2700 5400
+Wire Wire Line
+	2700 5400 2650 5400
+Wire Wire Line
+	3250 5100 3550 5100
+Wire Wire Line
+	3000 5100 3200 5100
+Wire Wire Line
+	3200 5100 3200 5200
+Wire Wire Line
+	3200 5200 3550 5200
+Wire Wire Line
+	2900 5400 3550 5400
+Wire Wire Line
+	3150 5150 3150 5350
+Wire Wire Line
+	3150 5350 3500 5350
+Wire Wire Line
+	3500 5350 3500 5300
+Wire Wire Line
+	3500 5300 3550 5300
 $Comp
 L power:+5V #PWR026
@@
 	7500 2550 7500 2400
 $Comp
-L Display_Character:SM420561N U2
-U 1 1 620F3E73
+L Display_Character:HDSP-A151 U2
+U 1 1 62073E2A
 P 3850 5100
 F 0 "U2" H 3850 5767 50  0000 C CNN
-F 1 "SM420561N" H 3850 5676 50  0000 C CNN
-F 2 "Display_7Segment:7SegmentLED_LTS6760_LTS6780" H 3900 4500 50  0001 C CNN
-F 3 "https://datasheet.lcsc.com/szlcsc/Wuxi-ARK-Tech-Elec-SM420561N_C141367.pdf" H 3350 5575 50  0001 L CNN
+F 1 "HDSP-A151" H 3850 5676 50  0000 C CNN
+F 2 "Display_7Segment:7SegmentLED_LTS6760_LTS6780" H 3850 4550 50  0001 C CNN
+F 3 "https://docs.broadcom.com/docs/AV02-2553EN" H 3350 5650 50  0001 C CNN
 	1    3850 5100
 	1    0    0    -1
 $EndComp
-NoConn ~ 1650 4850
-$Comp
-L 0805:R R10
-U 1 1 62556D66
-P 3150 1750
-F 0 "R10" H 3080 1704 50  0000 R CNN
-F 1 "10K" H 3080 1795 50  0000 R CNN
-F 2 "Resistor_SMD:R_0805_2012Metric" V 3080 1750 50  0001 C CNN
-F 3 "~" H 3150 1750 50  0001 C CNN
-	1    3150 1750
-	1    0    0    -1
-$EndComp
-$Comp
-L power:+5V #PWR029
-U 1 1 62557745
-P 3150 1450
-F 0 "#PWR029" H 3150 1300 50  0001 C CNN
-F 1 "+5V" H 3165 1623 50  0000 C CNN
-F 2 "" H 3150 1450 50  0001 C CNN
-F 3 "" H 3150 1450 50  0001 C CNN
-	1    3150 1450
-	1    0    0    -1
-$EndComp
-Wire Wire Line
-	3150 1450 3150 1600
-Wire Wire Line
-	3150 1900 3150 2100
-Connection ~ 3150 2100
-Wire Wire Line
-	3550 5500 3350 5500
-Wire Wire Line
-	3350 5500 3350 4800
-Wire Wire Line
-	3550 5000 2950 5000
-Wire Wire Line
-	2950 5000 2950 4900
-Wire Wire Line
-	2950 4900 2650 4900
-Wire Wire Line
-	2650 5000 2900 5000
-Wire Wire Line
-	2900 5000 2900 5100
-Wire Wire Line
-	2900 5100 3550 5100
-Wire Wire Line
-	3550 5200 2850 5200
-Wire Wire Line
-	2850 5200 2850 5100
-Wire Wire Line
-	2850 5100 2650 5100
-Wire Wire Line
-	2650 5300 3250 5300
-Wire Wire Line
-	3250 5300 3250 4900
-Wire Wire Line
-	3250 4900 3550 4900
-Wire Wire Line
-	3250 5500 3250 5450
-Wire Wire Line
-	3250 5450 3450 5450
-Wire Wire Line
-	3450 5450 3450 5300
-Wire Wire Line
-	3450 5300 3550 5300
-Wire Wire Line
-	2650 5500 3250 5500
-Wire Wire Line
-	3350 4800 2650 4800
-Wire Wire Line
-	3400 4800 3550 4800
-Wire Wire Line
-	2650 5400 3400 5400
-Wire Wire Line
-	3400 5400 3400 4800
-Wire Wire Line
-	3500 5650 2800 5650
-Wire Wire Line
-	2800 5650 2800 5200
-Wire Wire Line
-	2800 5200 2650 5200
-Wire Wire Line
-	3500 5650 3500 5400
-Wire Wire Line
-	3500 5400 3550 5400
+$Comp
+L Display_Character:SM420561N U?
+U 1 1 620F3E73
+P 4850 5050
+F 0 "U?" H 4850 5717 50  0000 C CNN
+F 1 "SM420561N" H 4850 5626 50  0000 C CNN
+F 2 "Display_7Segment:7SegmentLED_LTS6760_LTS6780" H 4900 4450 50  0001 C CNN
+F 3 "https://datasheet.lcsc.com/szlcsc/Wuxi-ARK-Tech-Elec-SM420561N_C141367.pdf" H 4350 5525 50  0001 L CNN
+	1    4850 5050
+	1    0    0    -1
+$EndComp
 $EndSCHEMATC
