File: V3/DB15_Switch/DB15_Switch/DB15_Switch_panelize.kicad_pcb (KiCad board)
At the start: 2 copper layers, 95.1 x 87.4 mm, 210 parts, among them J1 DB15_Male_HighDensity_Mountin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, U1 CH340C, U2 SM420561N, U3 STI3508, U4 ATmega328P-A, Y1 Crystal_GND24

Commit message: update
Other:
- net class Default removed
